File: mixed_signal_sensor_board.kicad_pcb (KiCad board)
At the start: 4 copper layers, 105.8 x 58 mm, 159 parts, among them J1 Conn_01x02, J10 Conn_01x04, J11 Conn_01x04, J12 Conn_01x04, J13 USB_C_Receptacle_USB2.0_16P, J14 Conn_01x04, J15 PYRO, J16 PYRO, J17 PYRO, J18 PYRO, J2 Conn_01x04, J3 Conn_01x06, J4 Conn_02x06_Odd_Even, J5 Conn_01x04, J6 Conn_01x04, J7 Conn_01x04, J8 Conn_01x04, J9 Conn_01x04, Q1 IRLML5103TRPBF, Q2 CSD17571Q2, Q3 CSD17571Q2, Q4 CSD17571Q2, Q5 CSD17571Q2, SW1 SW_Push, SW2 SW_Push, U1 TMP117xxDRV, U2 LM27762, U3 MagI3C_171013201, U4 TPS7A20xxxDBV, U5 TPS7A20xxxDBV, U6 ADS131M08xPBS, U7 STM32L552CEUx, U8 USBLC6-2P6, U9 TCAN3414DRBR, Y1 SG-8018CE_8.192M-TJHSA

Commit message: Compact board, Artistic Freedom
Parts:
- moved R12 80.0 mm to (191.9, 88.1)
- moved SW1 80.0 mm to (190.0, 85.6)
- moved C14 80.0 mm to (193.5, 87.6)
- moved SW2 75.7 mm to (182.4, 85.6)
- moved R13 74.6 mm to (184.2, 88.2), turned to 180 degrees
- moved J3 29.5 mm to (126.1, 76.2), turned to -90 degrees
- moved C11 28.6 mm to (146.4, 73.7), turned to 90 degrees
- moved R10 28.4 mm to (145.3, 72.2), turned to 90 degrees
- moved R9 26.0 mm to (145.3, 74.3), turned to 90 degrees
- moved J1 25.8 mm to (125.9, 93.0)
- moved C3 24.4 mm to (141.8, 71.4), turned to 0 degrees
- moved D1 21.3 mm to (132.6, 91.4), turned to 0 degrees
- moved U2 21.2 mm to (141.8, 73.6), turned to 90 degrees
- moved C6 20.6 mm to (143.1, 75.8), turned to 0 degrees
- moved R2 20.6 mm to (134.6, 91.4)
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Connections:
- J3 pad 1: +3V3 -> GND
- J3 pad 2: /CS -> /MOSI
- J3 pad 3: /SCLK -> /MISO
- J3 pad 4: /MISO -> /SCLK
- J3 pad 5: /MOSI -> /CS
- J3 pad 6: GND -> +3V3
Routing:
- net /USB_N: track 0.00 -> 31.4 mm
- net /USB_P: track 0.00 -> 30.8 mm
- net /PYRO4_FAULT: track 0.00 -> 26.4 mm
- net /PYRO4_SIGNAL: track 0.00 -> 24.4 mm
- net /PYRO1_FAULT: track 0.00 -> 18.9 mm
- net /SDA: track 0.00 -> 18.9 mm
- net /PYRO1_SIGNAL: track 0.00 -> 18.6 mm
- net /SCL: track 0.00 -> 16.4 mm
- net /CLK_IN: track 0.00 -> 14.3 mm
- net /PYRO3_FAULT: track 0.00 -> 13.4 mm
- net /ADS_SYNC/RESET: track 0.00 -> 13.2 mm
- net /ADS_DRDY: track 0.00 -> 12.2 mm
- net /PYRO3_SIGNAL: track 0.00 -> 11.2 mm
- net /LEDG: track 0.00 -> 10.9 mm
- net /LEDB: track 0.00 -> 10.4 mm
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Other:
- board size 105.8 x 58 mm -> 85 x 58 mm
- board text added: "+"
- board text added: "-"
- board text added: "DAQ PYRO CASTING CONTROLLER"
- board text added: "P02"
- board text added: "P03"
- board text added: "P04"
- board text added: "P12"
- board text added: "P25"
- board text added: "P26"
- board text added: "P27"
- board text added: "REV 1"
- board text added: "SB5"
- board text added: "SB6"
- board text removed: "PA2"
- board text removed: "PB12"
- board text removed: "PB13"
- board text removed: "PB14"
- board text removed: "PC13"
- board text removed: "PC14"
- board text removed: "PC15"

Commit message: Artistic Freedom
Parts:
- moved R14 1.25 mm to (202.0, 63.2)
- moved D3 1.25 mm to (202.0, 65.3)
- moved J4 0.50 mm to (192.1, 60.2)
- moved D1 0.40 mm to (132.9, 91.1)
- moved R2 0.40 mm to (134.9, 91.1)
- moved Q1 0.33 mm to (132.6, 88.8)
Other:
- board text added: "PYRO CASTING CONTROLLER"
- board text removed: "DAQ PYRO CASTING CONTROLLER"
